File: Power_Dist_Board/Power_Dist_Board.kicad_pcb (KiCad board)
At the start: 2 copper layers, 73 x 73 mm, 11 parts, among them P1 CONN_01X03, P10 CONN_02X04, P2 CONN_01X03, P3 CONN_01X03, P4 CONN_01X03, P5 CONN_01X03, P6 CONN_01X02, P7 CONN_01X02, P8 CONN_01X04, P9 CONN_02X08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

Commit message: Commit update
Parts:
- added C1: C, Capacitors_SMD:C_0805, F.Cu at (103.5, 106.2)
- added C2: C, Capacitors_SMD:C_0603, F.Cu at (110.2, 102.5)
- added C3: C, Capacitors_SMD:c_elec_6.3x4.5, F.Cu at (75.8, 105.2)
- added D1: LED, LEDs:LED_0805, F.Cu at (126.2, 98.0)
- added D2: LED, LEDs:LED_0805, F.Cu at (126.2, 103.5)
- added D3: LED, LEDs:LED_0805, F.Cu at (126.2, 100.8)
- added P11: CONN_01X03, Socket_Strips:Socket_Strip_Straight_1x03, B.Cu at (67.5, 107.3)
- added R1: R, Capacitors_SMD:C_0603, F.Cu at (121.2, 98.0)
- added R2: R, Capacitors_SMD:C_0603, F.Cu at (121.2, 103.5)
- added R3: R, Capacitors_SMD:C_0603, F.Cu at (121.2, 100.8)
- added U2: DSN-MINI-360, KiCad_Footprint:DSN-MINI-360, F.Cu at (91.8, 108.8)
- added U3: TLV1117LV33, TO_SOT_Packages_SMD:SOT-223, F.Cu at (109.0, 108.7)
- P10, P9: moved to B.Cu
- moved P8 11.2 mm to (96.2, 90.2)
- moved P6 10.8 mm to (93.8, 79.2)
- moved P7 10.8 mm to (103.8, 79.2)
- moved P1 5.01 mm to (104.8, 126.5), turned to 180 degrees
- moved P10 2.54 mm to (124.5, 85.5)
- moved P9 2.54 mm to (91.1, 73.0)
- moved P2 1.11 mm to (81.4, 79.2)
- moved P3 1.11 mm to (81.4, 90.2)
- moved U1 0.31 mm to (93.3, 100.0)
- moved P4 0.25 mm to (113.5, 79.2)
- moved P5 0.25 mm to (113.5, 90.2)
Connections:
- P10 pad 5: GND -> GNDPWR
- P10 pad 6: GND -> GNDPWR
- P10 pad 7: GND -> GNDPWR
- P10 pad 8: GND -> GNDPWR
- P2 pad 1: /Motor_1A -> /Motor_1C
- P2 pad 3: /Motor_1C -> /Motor_1A
- P3 pad 1: /Motor_2A -> /Motor_3A
- P3 pad 2: /Motor_2B -> /Motor_3B
- P3 pad 3: /Motor_2C -> /Motor_3C
- P4 pad 1: /Motor_3A -> /Motor_2C
- P4 pad 2: /Motor_3B -> /Motor_2B
- P4 pad 3: /Motor_3C -> /Motor_2A
- U1 pad C: (no net) -> Net-(R2-Pad1)
- U1 pad E: (no net) -> Net-(R3-Pad1)
- U1 pad P: (no net) -> Net-(R1-Pad1)
- U1 pad T_-: GND -> GNDPWR
Routing:
- net /Motor_1C: track 0.00 -> 26.0 mm
- net /Motor_2A: track 0.00 -> 25.7 mm
- net /Motor_3A: track 0.00 -> 22.3 mm
- net /Motor_3B: track 0.00 -> 21.8 mm
- net /Motor_4C: track 0.00 -> 21.8 mm
- net /Motor_3C: track 0.00 -> 21.3 mm
- net /Motor_4A: track 0.00 -> 21.2 mm
- net /Motor_4B: track 0.00 -> 21.2 mm
- net /SDA: track 0.00 -> 20.8 mm
- net /SCL: track 0.00 -> 20.8 mm
- net /Motor_1B: track 0.00 -> 19.2 mm
- net /Motor_2B: track 0.00 -> 18.8 mm
- net /Motor_1A: track 0.00 -> 11.4 mm
- net /Motor_2C: track 0.00 -> 10.7 mm
- net /LED-: track 0.00 -> 8.30 mm
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Other:
- outline, holes or cut-outs redrawn
- net class Default: trace_width 0.25 -> 0.3
