File: Power_Dist_Board/Power_Dist_Board.sch (KiCad schematic (older format))
At the start: 17 parts, among them P1 CONN_01X03, P10 CONN_02X04, P2 CONN_01X03, P3 CONN_01X03, P4 CONN_01X03, P5 CONN_01X03, P6 CONN_01X02, P7 CONN_01X02, P8 CONN_01X04, P9 CONN_02X08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

Commit message: Commit update
Parts:
- added C1: C, Capacitors_SMD:C_0805, symbol C
- added C2: C, Capacitors_SMD:C_0603, symbol C
- added C3: C, Capacitors_SMD:c_elec_6.3x4.5, symbol C
- added P11: CONN_01X03, Socket_Strips:Socket_Strip_Straight_1x03, symbol CONN_01X03
- added U2: DSN-MINI-360, KiCad_Footprint:DSN-MINI-360, symbol DSN-MINI-360
- added U3: TLV1117LV33, TO_SOT_Packages_SMD:SOT-223, symbol TLV1117LV33
- D1, D2, D3: footprint (none) -> LEDs:LED_0805
- R1, R2, R3: footprint (none) -> Capacitors_SMD:C_0603
Connections:
- net labels added: 5V, GNDPWR
- wire segments 66 -> 83
- no-connect marks 1 -> 2
Other:
- moved on the sheet: P3, P4
Changed lines of the file:
@@
 LIBS:valves
 LIBS:custom_lib
+LIBS:Power_Dist_Board-cache
 EELAYER 25 0
 EELAYER END
@@
 Wire Wire Line
 	10400 1325 10725 1325
-$Comp
-L GND #PWR02
-U 1 1 581D6F81
-P 10725 1325
-F 0 "#PWR02" H 10725 1075 50  0001 C CNN
-F 1 "GND" H 10725 1175 50  0000 C CNN
-F 2 "" H 10725 1325 50  0000 C CNN
-F 3 "" H 10725 1325 50  0000 C CNN
-	1    10725 1325
-	0    -1   -1   0
-$EndComp
 Wire Wire Line
 	8550 1125 7875 1125
@@
 F 0 "R1" V 8205 1525 50  0000 C CNN
 F 1 "R" V 8125 1525 50  0000 C CNN
-F 2 "" V 8055 1525 50  0000 C CNN
+F 2 "Capacitors_SMD:C_0603" V 8055 1525 50  0001 C CNN
 F 3 "" H 8125 1525 50  0000 C CNN
 	1    8125 1525
@@
 F 0 "R2" V 8205 1725 50  0000 C CNN
 F 1 "R" V 8125 1725 50  0000 C CNN
-F 2 "" V 8055 1725 50  0000 C CNN
+F 2 "Capacitors_SMD:C_0603" V 8055 1725 50  0001 C CNN
 F 3 "" H 8125 1725 50  0000 C CNN
 	1    8125 1725
@@
 F 0 "R3" V 8205 1925 50  0000 C CNN
 F 1 "R" V 8125 1925 50  0000 C CNN
-F 2 "" V 8055 1925 50  0000 C CNN
+F 2 "Capacitors_SMD:C_0603" V 8055 1925 50  0001 C CNN
 F 3 "" H 8125 1925 50  0000 C CNN
 	1    8125 1925
@@
 F 0 "D1" H 7650 1625 50  0000 C CNN
 F 1 "LED" H 7650 1425 50  0000 C CNN
-F 2 "" H 7650 1525 50  0000 C CNN
+F 2 "LEDs:LED_0805" H 7525 1650 50  0001 C CNN
 F 3 "" H 7650 1525 50  0000 C CNN
 	1    7650 1525
@@
 F 0 "D2" H 7650 1825 50  0000 C CNN
 F 1 "LED" H 7650 1625 50  0000 C CNN
-F 2 "" H 7650 1725 50  0000 C CNN
+F 2 "LEDs:LED_0805" H 6950 1775 50  0001 C CNN
 F 3 "" H 7650 1725 50  0000 C CNN
 	1    7650 1725
@@
 F 0 "D3" H 7650 2025 50  0000 C CNN
 F 1 "LED" H 7650 1825 50  0000 C CNN
-F 2 "" H 7650 1925 50  0000 C CNN
+F 2 "LEDs:LED_0805" H 7650 2125 50  0001 C CNB
 F 3 "" H 7650 1925 50  0000 C CNN
 	1    7650 1925
@@
 	7850 1925 7975 1925
 $Comp
-L GND #PWR03
+L GND #PWR02
 U 1 1 581D7652
 P 7325 1625
-F 0 "#PWR03" H 7325 1375 50  0001 C CNN
+F 0 "#PWR02" H 7325 1375 50  0001 C CNN
 F 1 "GND" H 7325 1475 50  0000 C CNN
 F 2 "" H 7325 1625 50  0000 C CNN
@@
 V_BAT+
 $Comp
-L GND #PWR04
+L GND #PWR03
 U 1 1 581D7B07
 P 1250 1050
-F 0 "#PWR04" H 1250 800 50  0001 C CNN
+F 0 "#PWR03" H 1250 800 50  0001 C CNN
 F 1 "GND" H 1250 900 50  0000 C CNN
 F 2 "" H 1250 1050 50  0000 C CNN
@@
 F 3 "" H 2050 1825 50  0000 C CNN
 	1    2050 1825
-	1    0    0    -1
+	1    0    0    1
 $EndComp
 Wire Wire Line
@@
 	3175 3000 2600 3000
 $Comp
-L GND #PWR05
+L GND #PWR04
 U 1 1 581D955A
 P 2600 3000
-F 0 "#PWR05" H 2600 2750 50  0001 C CNN
+F 0 "#PWR04" H 2600 2750 50  0001 C CNN
 F 1 "GND" H 2600 2850 50  0000 C CNN
 F 2 "" H 2600 3000 50  0000 C CNN
@@
 L CONN_01X03 P3
 U 1 1 581DF7FE
+P 2050 3025
+F 0 "P3" H 2050 3225 50  0000 C CNN
+F 1 "CONN_01X03" V 2150 3025 50  0000 C CNN
+F 2 "Connectors_JST:JST_XH_B03B-XH-A_03x2.50mm_Straight" H 2050 3025 50  0001 C CNN
+F 3 "" H 2050 3025 50  0000 C CNN
+	1    2050 3025
+	1    0    0    -1
+$EndComp
+$Comp
+L CONN_01X03 P4
+U 1 1 581DF84E
 P 2050 2425
-F 0 "P3" H 2050 2625 50  0000 C CNN
+F 0 "P4" H 2050 2625 50  0000 C CNN
 F 1 "CONN_01X03" V 2150 2425 50  0000 C CNN
 F 2 "Connectors_JST:JST_XH_B03B-XH-A_03x2.50mm_Straight" H 2050 2425 50  0001 C CNN
 F 3 "" H 2050 2425 50  0000 C CNN
 	1    2050 2425
-	1    0    0    -1
-$EndComp
-$Comp
-L CONN_01X03 P4
-U 1 1 581DF84E
-P 2050 3025
-F 0 "P4" H 2050 3225 50  0000 C CNN
-F 1 "CONN_01X03" V 2150 3025 50  0000 C CNN
-F 2 "Connectors_JST:JST_XH_B03B-XH-A_03x2.50mm_Straight" H 2050 3025 50  0001 C CNN
-F 3 "" H 2050 3025 50  0000 C CNN
-	1    2050 3025
-	1    0    0    -1
+	1    0    0    1
 $EndComp
 $Comp
@@
 Text Label 5550 2425 0    60   ~ 0
 V_BAT+
-$Comp
-L GND #PWR06
-U 1 1 581E142B
-P 4475 2625
-F 0 "#PWR06" H 4475 2375 50  0001 C CNN
-F 1 "GND" H 4475 2475 50  0000 C CNN
-F 2 "" H 4475 2625 50  0000 C CNN
-F 3 "" H 4475 2625 50  0000 C CNN
-	1    4475 2625
-	0    1    1    0
-$EndComp
 Wire Wire Line
 	4475 2625 4875 2625
@@
 	4725 2725 4725 2625
 Connection ~ 4725 2625
+Wire Wire Line
+	5375 2625 5750 2625
+Wire Wire Line
+	5375 2725 5550 2725
+Wire Wire Line
+	5550 2725 5550 2625
+Connection ~ 5550 2625
+$Comp
+L DSN-MINI-360 U2
+U 1 1 581D2956
+P 8775 2700
+F 0 "U2" H 9025 2500 60  0000 C CNN
+F 1 "DSN-MINI-360" H 8775 2875 43  0000 C CNN
+F 2 "KiCad_Footprint:DSN-MINI-360" H 8700 2525 60  0001 C CNN
+F 3 "" H 8700 2525 60  0001 C CNN
+	1    8775 2700
+	1    0    0    -1
+$EndComp
+Wire Wire Line
+	8250 2725 8125 2725
+Wire Wire Line
+	8125 2725 8125 2825
+Wire Wire Line
+	8250 2625 7675 2625
+Text Label 7675 2625 0    60   ~ 0
+V_BAT+
+Wire Wire Line
+	9300 2625 9950 2625
+$Comp
+L GND #PWR05
+U 1 1 581D3E8C
+P 9475 3050
+F 0 "#PWR05" H 9475 2800 50  0001 C CNN
+F 1 "GND" H 9475 2900 50  0000 C CNN
+F 2 "" H 9475 3050 50  0000 C CNN
+F 3 "" H 9475 3050 50  0000 C CNN
+	1    9475 3050
+	1    0    0    -1
+$EndComp
+Wire Wire Line
+	9300 2725 9475 2725
+Wire Wire Line
+	9475 2725 9475 3050
+Text Label 9850 2625 0    60   ~ 0
+5V
+$Comp
+L CONN_01X03 P11
+U 1 1 581D4605
+P 3375 3900
+F 0 "P11" H 3375 4100 50  0000 C CNN
+F 1 "CONN_01X03" V 3475 3900 50  0000 C CNN
+F 2 "Socket_Strips:Socket_Strip_Straight_1x03" H 3375 3900 50  0001 C CNN
+F 3 "" H 3375 3900 50  0000 C CNN
+	1    3375 3900
+	1    0    0    1
+$EndComp
+Wire Wire Line
+	3175 3800 2600 3800
+Wire Wire Line
+	3175 4000 2700 4000
+$Comp
+L GND #PWR06
+U 1 1 581D49C2
+P 2700 4000
+F 0 "#PWR06" H 2700 3750 50  0001 C CNN
+F 1 "GND" H 2700 3850 50  0000 C CNN
+F 2 "" H 2700 4000 50  0000 C CNN
+F 3 "" H 2700 4000 50  0000 C CNN
+	1    2700 4000
+	0    1    1    0
+$EndComp
+Text Label 2600 3800 0    60   ~ 0
+5V
+NoConn ~ 3175 3900
+$Comp
+L TLV1117LV33 U3
+U 1 1 581D4F7C
+P 8775 3600
+F 0 "U3" H 8475 3850 50  0000 C CNN
+F 1 "TLV1117LV33" H 8775 3800 50  0000 C CNN
+F 2 "TO_SOT_Packages_SMD:SOT-223" H 8775 3700 50  0001 C CIN
+F 3 "" H 8775 3600 50  0000 C CNN
+	1    8775 3600
+	1    0    0    -1
+$EndComp
 $Comp
 L GND #PWR07
-U 1 1 581E1516
+U 1 1 581D53D0
+P 8775 4050
+F 0 "#PWR07" H 8775 3800 50  0001 C CNN
+F 1 "GND" H 8775 3900 50  0000 C CNN
+F 2 "" H 8775 4050 50  0000 C CNN
+F 3 "" H 8775 4050 50  0000 C CNN
+	1    8775 4050
+	1    0    0    -1
+$EndComp
+Wire Wire Line
+	8775 3900 8775 4050
+Wire Wire Line
+	8325 3550 7725 3550
+Text Label 7725 3550 0    60   ~ 0
+5V
+Wire Wire Line
+	9225 3550 9950 3550
+Wire Wire Line
+	9225 3700 9325 3700
+Wire Wire Line
+	9325 3700 9325 3550
+Connection ~ 9325 3550
+Text Label 9775 3550 0    60   ~ 0
+3V3
+$Comp
+L C C1
+U 1 1 581DDF64
+P 8050 3700
+F 0 "C1" H 8075 3800 50  0000 L CNN
+F 1 "C" H 8075 3600 50  0000 L CNN
+F 2 "Capacitors_SMD:C_0805" H 8088 3550 50  0001 C CNN
+F 3 "" H 8050 3700 50  0000 C CNN
+	1    8050 3700
+	1    0    0    -1
+$EndComp
+Wire Wire Line
+	8050 4000 9525 4000
+Wire Wire Line
+	8050 4000 8050 3850
+Connection ~ 8775 4000
+Connection ~ 8050 3550
+$Comp
+L C C2
+U 1 1 581DE06E
+P 9525 3700
+F 0 "C2" H 9550 3800 50  0000 L CNN
+F 1 "C" H 9550 3600 50  0000 L CNN
+F 2 "Capacitors_SMD:C_0603" H 9563 3550 50  0001 C CNN
+F 3 "" H 9525 3700 50  0000 C CNN
+	1    9525 3700
+	1    0    0    -1
+$EndComp
+Wire Wire Line
+	9525 4000 9525 3850
+Connection ~ 9525 3550
+$Comp
+L GNDPWR #PWR08
+U 1 1 581DEDA7
+P 4475 2625
+F 0 "#PWR08" H 4475 2425 50  0001 C CNN
+F 1 "GNDPWR" H 4475 2495 50  0000 C CNN
+F 2 "" H 4475 2575 50  0000 C CNN
+F 3 "" H 4475 2575 50  0000 C CNN
+	1    4475 2625
+	0    1    1    0
+$EndComp
+$Comp
+L GNDPWR #PWR09
+U 1 1 581DF5F0
 P 5750 2625
-F 0 "#PWR07" H 5750 2375 50  0001 C CNN
-F 1 "GND" H 5750 2475 50  0000 C CNN
-F 2 "" H 5750 2625 50  0000 C CNN
-F 3 "" H 5750 2625 50  0000 C CNN
+F 0 "#PWR09" H 5750 2425 50  0001 C CNN
+F 1 "GNDPWR" H 5750 2495 50  0000 C CNN
+F 2 "" H 5750 2575 50  0000 C CNN
+F 3 "" H 5750 2575 50  0000 C CNN
 	1    5750 2625
 	0    -1   -1   0
 $EndComp
-Wire Wire Line
-	5375 2625 5750 2625
-Wire Wire Line
-	5375 2725 5550 2725
-Wire Wire Line
-	5550 2725 5550 2625
-Connection ~ 5550 2625
+$Comp
+L GNDPWR #PWR010
+U 1 1 581DFF23
+P 8125 2825
+F 0 "#PWR010" H 8125 2625 50  0001 C CNN
+F 1 "GNDPWR" H 8125 2695 50  0000 C CNN
+F 2 "" H 8125 2775 50  0000 C CNN
+F 3 "" H 8125 2775 50  0000 C CNN
+	1    8125 2825
+	1    0    0    -1
+$EndComp
+$Comp
+L GNDPWR #PWR011
+U 1 1 581E0462
+P 10725 1325
+F 0 "#PWR011" H 10725 1125 50  0001 C CNN
+F 1 "GNDPWR" H 10725 1195 50  0000 C CNN
+F 2 "" H 10725 1275 50  0000 C CNN
+F 3 "" H 10725 1275 50  0000 C CNN
+	1    10725 1325
+	0    -1   -1   0
+$EndComp
+$Comp
+L C C3
+U 1 1 581E1529
+P 9775 2775
+F 0 "C3" H 9800 2875 50  0000 L CNN
+F 1 "C" H 9800 2675 50  0000 L CNN
+F 2 "Capacitors_SMD:c_elec_6.3x4.5" H 9813 2625 50  0001 C CNN
+F 3 "" H 9775 2775 50  0000 C CNN
+	1    9775 2775
+	1    0    0    -1
+$EndComp
+Connection ~ 9775 2625
+Wire Wire Line
+	9775 2925 9475 2925
+Connection ~ 9475 2925
 $EndSCHEMATC
