File: ESC_Module/ESC_Module.sch (KiCad schematic (older format))
At the start: 3 parts, among them P1 CONN_02X04, P2 CONN_02X04, U1 DYS_mini_ESC

Commit message: modify..
Parts:
- added C1: 330uF, Capacitors_SMD:c_elec_8x10, symbol CP1
Connections:
- wire segments 21 -> 23
Changed lines of the file:
@@
 V_BAT
 Wire Wire Line
-	1700 1050 2250 1050
+	1700 1050 2900 1050
 Text Label 2000 1050 0    60   ~ 0
 V_BAT
 $Comp
-L GND #PWR01
+L GND #PWR1
 U 1 1 580215D7
 P 825 1200
-F 0 "#PWR01" H 825 950 50  0001 C CNN
+F 0 "#PWR1" H 825 950 50  0001 C CNN
 F 1 "GND" H 825 1050 50  0000 C CNN
 F 2 "" H 825 1200 50  0000 C CNN
@@
 Connection ~ 825  1200
 $Comp
-L GND #PWR02
+L GND #PWR2
 U 1 1 58021605
 P 2150 1200
-F 0 "#PWR02" H 2150 950 50  0001 C CNN
+F 0 "#PWR2" H 2150 950 50  0001 C CNN
 F 1 "GND" H 2150 1050 50  0000 C CNN
 F 2 "" H 2150 1200 50  0000 C CNN
@@
 $EndComp
 $Comp
-L GND #PWR03
+L GND #PWR4
 U 1 1 580237F7
 P 4175 1825
-F 0 "#PWR03" H 4175 1575 50  0001 C CNN
+F 0 "#PWR4" H 4175 1575 50  0001 C CNN
 F 1 "GND" H 4175 1675 50  0000 C CNN
 F 2 "" H 4175 1825 50  0000 C CNN
@@
 Text Label 3825 1975 0    60   ~ 0
 PWM_Input
+$Comp
+L CP1 C1
+U 1 1 5820023A
+P 2625 1250
+F 0 "C1" H 2650 1350 50  0000 L CNN
+F 1 "330uF" H 2650 1150 50  0000 L CNN
+F 2 "Capacitors_SMD:c_elec_8x10" H 2625 1250 50  0001 C CNN
+F 3 "" H 2625 1250 50  0000 C CNN
+	1    2625 1250
+	1    0    0    -1
+$EndComp
+Wire Wire Line
+	2625 1050 2625 1100
+Connection ~ 2625 1050
+$Comp
+L GND #PWR3
+U 1 1 5820029B
+P 2625 1475
+F 0 "#PWR3" H 2625 1225 50  0001 C CNN
+F 1 "GND" H 2625 1325 50  0000 C CNN
+F 2 "" H 2625 1475 50  0000 C CNN
+F 3 "" H 2625 1475 50  0000 C CNN
+	1    2625 1475
+	1    0    0    -1
+$EndComp
+Wire Wire Line
+	2625 1400 2625 1475
 $EndSCHEMATC
