File: LED_Module/LED_Module.kicad_pcb (KiCad board)
At the start: 2 copper layers, 25 x 25 mm, 13 parts, among them P1 CONN_01X01, P2 CONN_01X01, P3 CONN_01X01, P4 CONN_01X01, P5 CONN_01X01, U1 AL8805WS

Commit message: LED Module PWM pull down
Parts:
- added R2: 10k, Resistors_SMD:R_0805_HandSoldering, F.Cu at (93.5, 91.5)
Changed lines of the file:
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@@
 (kicad_pcb (version 4) (host pcbnew 4.0.4-stable)
   (general
-    (links 18)
+    (links 20)
     (no_connects 0)
     (area 87.424999 87.424999 112.575001 112.575001)
     (thickness 1.6)
     (drawings 13)
-    (tracks 49)
+    (tracks 50)
     (zones 0)
-    (modules 13)
+    (modules 14)
     (nets 7)
   )
@@
     (last_trace_width 0.7)
     (trace_clearance 0.2)
-    (zone_clearance 0.2)
+    (zone_clearance 0.508)
     (zone_45_only no)
     (trace_min 0.2)
@@
       (net 5 /LED1-))
   )
+  (module Resistors_SMD:R_0805_HandSoldering (layer F.Cu)
+    (at 93.5 91.5 90)
+    (descr "Resistor SMD 0805, hand soldering")
+    (tags "resistor 0805")
+    (attr smd)
+    (fp_text reference R2 (at 0 -2.1 90) (layer F.SilkS) hide
+      (effects (font (size 1 1) (thickness 0.15)))
+    )
+    (fp_text value 10k (at 0 2.1 90) (layer F.Fab)
+      (effects (font (size 1 1) (thickness 0.15)))
+    )
+    (fp_line (start -2.4 -1) (end 2.4 -1) (layer F.CrtYd) (width 0.05))
+    (fp_line (start -2.4 1) (end 2.4 1) (layer F.CrtYd) (width 0.05))
+    (fp_line (start -2.4 -1) (end -2.4 1) (layer F.CrtYd) (width 0.05))
+    (fp_line (start 2.4 -1) (end 2.4 1) (layer F.CrtYd) (width 0.05))
+    (fp_line (start 0.6 0.875) (end -0.6 0.875) (layer F.SilkS) (width 0.15))
+    (fp_line (start -0.6 -0.875) (end 0.6 -0.875) (layer F.SilkS) (width 0.15))
+    (pad 1 smd rect (at -1.35 0 90) (size 1.5 1.3) (layers F.Cu F.Paste F.Mask)
+      (net 3 /CTRL_PWM))
+    (pad 2 smd rect (at 1.35 0 90) (size 1.5 1.3) (layers F.Cu F.Paste F.Mask)
+      (net 1 GND))
+    (model Resistors_SMD.3dshapes/R_0805_HandSoldering.wrl
+      (at (xyz 0 0 0))
+      (scale (xyz 1 1 1))
+      (rotate (xyz 0 0 0))
+    )
+  )
   (gr_line (start 91.5 102.5) (end 91.5 112.5) (layer Edge.Cuts) (width 0.15))
   (gr_line (start 87.5 102.5) (end 91.5 102.5) (layer Edge.Cuts) (width 0.15))
@@
   (via (at 98.6 101) (size 0.6) (drill 0.4) (layers F.Cu B.Cu) (net 1))
   (segment (start 102.7 109.25) (end 103.4 109.25) (width 0.5) (layer F.Cu) (net 1))
-  (segment (start 92.436 94) (end 93.49264 92.94336) (width 0.5) (layer F.Cu) (net 3))
-  (segment (start 93.49264 92.94336) (end 95.5475 92.94336) (width 0.5) (layer F.Cu) (net 3))
-  (segment (start 89.75 94) (end 92.436 94) (width 0.5) (layer F.Cu) (net 3))
+  (segment (start 93.5 92.85) (end 95.45414 92.85) (width 0.7) (layer F.Cu) (net 3))
+  (segment (start 95.45414 92.85) (end 95.5475 92.94336) (width 0.7) (layer F.Cu) (net 3))
+  (segment (start 89.75 94) (end 92.35 94) (width 0.7) (layer F.Cu) (net 3))
+  (segment (start 92.35 94) (end 93.5 92.85) (width 0.7) (layer F.Cu) (net 3))
   (segment (start 100 104.9) (end 100 105.7) (width 0.5) (layer B.Cu) (net 4))
   (via (at 100 105.7) (size 0.6) (drill 0.4) (layers F.Cu B.Cu) (net 4))
@@
     (polygon
       (pts
-        (xy 97.1 92) (xy 97.1 93.8) (xy 100.6 93.8) (xy 100.9 94.2) (xy 100.9 97.4)
-        (xy 107.442 97.409) (xy 108.712 96.139) (xy 108.7 92)
+        (xy 97.3 92.1) (xy 97.3 93.7) (xy 100.6 93.7) (xy 100.9 94.2) (xy 100.9 97.4)
+        (xy 107.442 97.409) (xy 108.8 96.1) (xy 108.8 92.1)
       )
     )
@@
   )
   (zone (net 1) (net_name GND) (layer F.Cu) (hatch edge 0.508)
-    (connect_pads (clearance 0.508))
-    (min_thickness 0.254)
-    (fill yes (arc_segments 16) (thermal_gap 0.508) (thermal_bridge_width 0.508))
-    (polygon
-      (pts
-        (xy 95.3 88.1) (xy 99.5 88.1) (xy 99.5 91.4) (xy 95.3 91.4)
-      )
-    )
+    (connect_pads yes (clearance 0.508))
+    (min_thickness 0.254)
+    (fill yes (arc_segments 16) (thermal_gap 0.508) (thermal_bridge_width 0.508))
+    (polygon
+      (pts
+        (xy 92.5 88) (xy 99.5 88) (xy 99.5 91.5) (xy 92.5 91.5)
+      )
+    )
