File: USB_Dist_Board/Maple_mini.sch (KiCad schematic (older format))
At the start: 22 parts, among them P2 CONN_01X03, Q1 BSS84, SW1 RESET, SW2 BOOT, U2 STM32F103CBT6, X1 8.000Mhz

Commit message: USB_Dist_Board change pin map
Parts:
- R11, R12, R3, R4, R5, R8, R9: footprint Resistors_SMD:R_0603 -> Capacitors_SMD:C_0603
Connections:
- net labels removed: ADC1
- wire segments 67 -> 66
Changed lines of the file:
@@
 F 0 "R8" V 2555 1825 50  0000 C CNN
 F 1 "10k" V 2475 1825 50  0000 C CNN
-F 2 "Resistors_SMD:R_0603" V 2405 1825 50  0001 C CNN
+F 2 "Capacitors_SMD:C_0603" V 2405 1825 50  0001 C CNN
 F 3 "" H 2475 1825 50  0000 C CNN
 	1    2475 1825
@@
 F 0 "R4" V 1780 4400 50  0000 C CNN
 F 1 "330" V 1700 4400 50  0000 C CNN
-F 2 "Resistors_SMD:R_0603" V 1630 4400 50  0001 C CNN
+F 2 "Capacitors_SMD:C_0603" V 1630 4400 50  0001 C CNN
 F 3 "" H 1700 4400 50  0000 C CNN
 	1    1700 4400
@@
 F 0 "R11" V 10450 4650 50  0000 C CNN
 F 1 "22" V 10525 4650 50  0000 C CNN
-F 2 "Resistors_SMD:R_0603" V 10455 4650 50  0001 C CNN
+F 2 "Capacitors_SMD:C_0603" V 10455 4650 50  0001 C CNN
 F 3 "" H 10525 4650 50  0000 C CNN
 	1    10525 4650
@@
 F 0 "R12" V 10625 4750 50  0000 C CNN
 F 1 "22" V 10525 4750 50  0000 C CNN
-F 2 "Resistors_SMD:R_0603" V 10455 4750 50  0001 C CNN
+F 2 "Capacitors_SMD:C_0603" V 10455 4750 50  0001 C CNN
 F 3 "" H 10525 4750 50  0000 C CNN
 	1    10525 4750
@@
 F 0 "R9" V 2755 1825 50  0000 C CNN
 F 1 "10k" V 2675 1825 50  0000 C CNN
-F 2 "Resistors_SMD:R_0603" V 2605 1825 50  0001 C CNN
+F 2 "Capacitors_SMD:C_0603" V 2605 1825 50  0001 C CNN
 F 3 "" H 2675 1825 50  0000 C CNN
 	1    2675 1825
@@
 Text HLabel 9325 4550 2    60   Input ~ 0
 PWM6
-Text HLabel 9150 3950 2    60   Input ~ 0
-ADC1
 Text HLabel 6050 1600 3    60   Input ~ 0
 GND
@@
 F 0 "R5" V 9630 4900 50  0000 C CNN
 F 1 "1.5k" V 9550 4900 50  0000 C CNN
-F 2 "Resistors_SMD:R_0603" V 9480 4900 50  0001 C CNN
+F 2 "Capacitors_SMD:C_0603" V 9480 4900 50  0001 C CNN
 F 3 "" H 9550 4900 50  0000 C CNN
 	1    9550 4900
@@
 F 0 "R3" V 9105 5700 50  0000 C CNN
 F 1 "10k" V 9025 5700 50  0000 C CNN
-F 2 "Resistors_SMD:R_0603" V 8955 5700 50  0001 C CNN
+F 2 "Capacitors_SMD:C_0603" V 8955 5700 50  0001 C CNN
 F 3 "" H 9025 5700 50  0000 C CNN
 	1    9025 5700
@@
 	8700 4550 9325 4550
 Wire Wire Line
-	8700 3950 9150 3950
-Wire Wire Line
 	6050 1275 6050 1600
