File: USB_Dist_Board/Maple_mini_2.sch (KiCad schematic (older format))
At the start: 22 parts, among them P2 CONN_01X03, Q3 BSS84, SW1 RESET, SW2 BOOT, U2 STM32F103CBT6, X1 8.000Mhz

Commit message: Add Power Distribution Board
Changed lines of the file:
@@
 Text HLabel 10250 3575 0    60   Input ~ 0
 GND
-Text HLabel 2225 4150 0    60   Input ~ 0
+Text HLabel 2225 4550 0    60   Input ~ 0
 I2C_SCL
-Text HLabel 2225 4250 0    60   Input ~ 0
+Text HLabel 2225 4650 0    60   Input ~ 0
 I2C_SDA
 $Comp
@@
 	10600 4750 10975 4750
 Wire Wire Line
-	2900 4150 2225 4150
-Wire Wire Line
-	2900 4250 2225 4250
-Wire Wire Line
 	8975 6025 9500 6025
 Connection ~ 9500 6025
+Wire Wire Line
+	2900 4550 2225 4550
+Wire Wire Line
+	2900 4650 2225 4650
 $EndSCHEMATC

Commit message: USB_Dist_Board change pin map
Parts:
- removed SW2: BOOT, Socket_Strips:Socket_Strip_Straight_1x02, symbol CONN_01X02
- R11, R12, R13, R15, R4, R8, R9: footprint Resistors_SMD:R_0603 -> Capacitors_SMD:C_0603
Connections:
- net labels added: ADC1, BOOT, PWR_SW
- wire segments 65 -> 66
