File: USB_Dist_Board/USB_Dist_Board.sch (KiCad schematic (older format))
At the start: 16 parts, among them P1 CONN_02X06, P5 CONN_01X04, P6 CONN_01X04, P7 CONN_02X06, U1 Raspberry_Front, U4 MCP1703T-3302E, U5 MCP1703T-3302E

Commit message: Add Power Distribution Board
Connections:
- wire segments 99 -> 98
Changed lines of the file:
@@
 Text Label 950  4975 0    60   ~ 0
 SDA
-Text Label 2975 4725 0    60   ~ 0
-USB_B_GND
 $Comp
 L CONN_01X04 P5
@@
 	9000 6200 8300 6200
 Wire Wire Line
-	950  4425 3575 4425
-Wire Wire Line
 	9000 3975 8300 3975
 Wire Wire Line
@@
 	1775 4875 1775 5100
 Connection ~ 1775 5100
-Wire Wire Line
-	3575 4725 2975 4725
 Wire Wire Line
 	1325 5875 1975 5875
@@
 	-1   0    0    1
 $EndComp
+Wire Wire Line
+	950  4425 2150 4425
 $EndSCHEMATC

Commit message: USB_Dist_Board change pin map
Parts:
- removed C1: C, Capacitors_SMD:C_0805, symbol C
- removed R23, R24: R, Resistors_SMD:R_0603, symbol R
- added R6: R, Capacitors_SMD:C_0603, symbol R
- P1, P7: value CONN_02X06 -> CONN_02X04; footprint Socket_Strips:Socket_Strip_Straight_2x06 -> Socket_Strips:Socket_Strip_Straight_2x04; symbol CONN_02X06 -> CONN_02X04
- R1: value 3.3k -> R; footprint Resistors_SMD:R_0603 -> Capacitors_SMD:C_0603
- R2: value 16.7k -> R; footprint Resistors_SMD:R_0603 -> Capacitors_SMD:C_0603
Connections:
- net labels added: BOOT, PWR_SW
- net labels removed: VCC_Bat
- wire segments 98 -> 86
Other:
- note removed: "20V full sacle to 3.3V ADC"
- moved on the sheet: P5, P6

Commit message: Main Board incomplete routing
Connections:
- wire segments 86 -> 85
- no-connect marks 0 -> 1
Changed lines of the file:
@@
 Text Label 1075 3075 0    60   ~ 0
-USB_D_GND
-Text Label 2225 3075 0    60   ~ 0
 USB_D_GND
 $Comp
@@
 	1075 3075 1575 3075
 Wire Wire Line
-	2075 3075 2725 3075
-Wire Wire Line
 	3200 1875 3800 1875
 Wire Wire Line
@@
 Text Label 2250 3900 0    60   ~ 0
 USB_B_GND
+NoConn ~ 2075 3075
 $EndSCHEMATC

Commit message: Main Board : Recover LED driver USB Dist Board : Delete ADC voltage divider
Parts:
- removed R1, R2: R, Capacitors_SMD:C_0603, symbol R
Connections:
- wire segments 85 -> 82
Changed lines of the file:
@@
 Text Label 1050 4200 0    60   ~ 0
 USB_B_GND
-Text Label 2550 4575 0    60   ~ 0
+Text Label 2550 4200 0    60   ~ 0
 ADC1
 Text Label 1050 4100 0    60   ~ 0
@@
 Text Label 8300 4900 0    60   ~ 0
 PWR_SW
-$Comp
-L R R1
-U 1 1 582B2ECF
-P 2275 4350
-F 0 "R1" V 2355 4350 50  0000 C CNN
-F 1 "R" V 2275 4350 50  0000 C CNN
-F 2 "Capacitors_SMD:C_0603" V 2205 4350 50  0001 C CNN
-F 3 "" H 2275 4350 50  0000 C CNN
-	1    2275 4350
-	1    0    0    -1
-$EndComp
-Text Label 2275 5025 3    60   ~ 0
-USB_B_GND
-$Comp
-L R R2
-U 1 1 582B441F
-P 2275 4800
-F 0 "R2" V 2355 4800 50  0000 C CNN
-F 1 "R" V 2275 4800 50  0000 C CNN
-F 2 "Capacitors_SMD:C_0603" V 2205 4800 50  0001 C CNN
-F 3 "" H 2275 4800 50  0000 C CNN
-	1    2275 4800
-	1    0    0    -1
-$EndComp
 $Comp
 L R R6
@@
 	9000 4900 8300 4900
 Wire Wire Line
-	2275 4500 2275 4650
-Wire Wire Line
-	2275 4950 2275 5525
-Wire Wire Line
-	2275 4575 2750 4575
-Connection ~ 2275 4575
-Wire Wire Line
-	2075 4200 2275 4200
-Wire Wire Line
 	950  4000 950  4200
 Connection ~ 950  4000
@@
 USB_B_GND
 NoConn ~ 2075 3075
+Wire Wire Line
+	2075 4200 2775 4200
 $EndSCHEMATC
