File: Main_Board/Main_Board.kicad_pcb (KiCad board)
At the start: 2 copper layers, 99 x 70 mm, 89 parts, among them J1 DB25, P1 CONN_01X06, P10 CONN_01X02, P11 CONN_01X02, P12 CONN_01X02, P13 CONN_02X07, P14 USB_A, P2 CONN_01X06, P3 CONN_01X03, P4 CONN_01X02, P5 CONN_01X02, P6 BOOT, P7 CONN_01X06, P8 CONN_01X04, P9 CONN_01X02, Q1 DMN65D8L, Q2 BSS84, Q3 BSS138, Q4 BSS138, SW1 RESET, U1 TLV1117LV33, U10 DSN-MINI-360, U11 TLV1117LV33, U12 STM32F103CBT6, U13 pca9685, U2 DYS_mini_ESC, U3 DYS_mini_ESC, U4 DYS_mini_ESC, U5 DYS_mini_ESC, U6 TENDA_P200, U7 AL8805W5, U8 AL8805W5, U9 SI4425DDY, X1 8MHz

Commit message: Final Routing
Parts:
- removed P5: CONN_01X02, Socket_Strips:Socket_Strip_Straight_1x02
- added C22: 10nF, Capacitors_SMD:C_0603, F.Cu at (232.4, 81.5)
- added C23: 0.1uF, Capacitors_SMD:C_0603, F.Cu at (232.4, 79.8)
- added C24: 0.1uF, Capacitors_SMD:C_0603, F.Cu at (232.4, 78.2)
- added P15: CONN_01X07, Socket_Strips:Socket_Strip_Straight_1x07, F.Cu at (53.0, 71.0)
- added P16: CONN_01X03, Socket_Strips:Socket_Strip_Straight_1x03, F.Cu at (232.0, 129.0)
- added P17: CONN_01X03, Socket_Strips:Socket_Strip_Straight_1x03, F.Cu at (122.0, 129.0)
- added U14: MPU9250, Housings_DFN_QFN:QFN-24-1EP_3x3mm_Pitch0.4mm, F.Cu at (227.6, 79.8)
- P1, P2, P7: value CONN_01X06 -> CONN_01X04; footprint Socket_Strips:Socket_Strip_Straight_1x06 -> Socket_Strips:Socket_Strip_Straight_1x04
- P11, P12: value CONN_01X02 -> CONN_01X03; footprint Socket_Strips:Socket_Strip_Straight_1x02 -> Socket_Strips:Socket_Strip_Straight_1x03
- P13: value CONN_02X07 -> CONN_01X07; footprint Socket_Strips:Socket_Strip_Straight_2x07 -> Socket_Strips:Socket_Strip_Straight_1x07
- P14: value USB_A -> CONN_01X04; footprint Connect:USB_Mini-B -> Connectors_Molex:Molex_PicoBlade_53047-0410_04x1.25mm_Straight
- moved P14 176.5 mm to (227.8, 89.2)
- moved Q4 172.6 mm to (229.6, 70.3)
- moved R17 172.6 mm to (227.1, 70.3)
- moved R16 172.6 mm to (232.2, 70.3)
- moved Q3 172.5 mm to (229.6, 74.1)
- moved R14 172.5 mm to (232.3, 74.1)
- moved R15 172.4 mm to (227.0, 74.1)
- moved R22 139.3 mm to (212.9, 99.4)
- moved R21 139.3 mm to (215.5, 96.8)
- moved Q2 139.3 mm to (215.5, 99.4)
- moved R24 139.2 mm to (211.2, 99.4)
- moved C20 139.2 mm to (211.9, 96.8)
- moved C14 139.2 mm to (211.6, 81.6)
- moved R23 139.2 mm to (209.4, 99.4)
- moved C19 139.2 mm to (208.7, 96.8)
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Connections:
- net /3V3 renamed /Upper_Board/3V3_PLC
- net /Bottom_Board/BOOT0 renamed /Upper_Board/BOOT0
- net /Bottom_Board/DISC renamed /Upper_Board/DISC
- net /Bottom_Board/OSC_IN renamed /Upper_Board/OSC_IN
- net /Bottom_Board/OSC_OUT renamed /Upper_Board/OSC_OUT
- net /Bottom_Board/SCL_5V renamed /Upper_Board/SCL_5V
- net /Bottom_Board/SDA_5V renamed /Upper_Board/SDA_5V
- net /Bottom_Board/USBDM renamed /Upper_Board/USBDM
- net /Bottom_Board/USBDP renamed /Upper_Board/USBDP
- C1 pad 1: /5V -> /Upper_Board/5V
- C1 pad 2: GND -> /Upper_Board/U_GND
- C11 pad 1: /Bottom_Board/5V -> /Upper_Board/5V
- C11 pad 2: GNDD -> /Upper_Board/U_GND
- C12 pad 1: /Bottom_Board/3V3 -> /Upper_Board/3V3
- C12 pad 2: GNDD -> /Upper_Board/U_GND
- C13 pad 2: GNDD -> /Upper_Board/U_GND
- C14 pad 2: GNDD -> /Upper_Board/U_GND
- C15 pad 1: /Bottom_Board/3V3 -> /Upper_Board/3V3
- C15 pad 2: GNDD -> /Upper_Board/U_GND
- C16 pad 1: /Bottom_Board/3V3 -> /Upper_Board/3V3
- C16 pad 2: GNDD -> /Upper_Board/U_GND
- C17 pad 1: /Bottom_Board/3V3 -> /Upper_Board/3V3
- C17 pad 2: GNDD -> /Upper_Board/U_GND
- C18 pad 1: /Bottom_Board/3V3 -> /Upper_Board/3V3
- C18 pad 2: GNDD -> /Upper_Board/U_GND
- C19 pad 2: GNDD -> /Upper_Board/U_GND
- C2 pad 2: GND -> /Upper_Board/U_GND
- C20 pad 2: GNDD -> /Upper_Board/U_GND
- C21 pad 1: /Bottom_Board/5V -> /Upper_Board/5V
- C21 pad 2: GNDD -> /Upper_Board/U_GND
- D1 pad 1: GND -> /Upper_Board/U_GND
- J1 pad 1: (no net) -> /Bottom_Board/V_BAT
- J1 pad 10: (no net) -> /Bottom_Board/MOTOR_4A
- J1 pad 11: (no net) -> /Bottom_Board/MOTOR_3C
- J1 pad 12: (no net) -> /Bottom_Board/MOTOR_3B
- J1 pad 13: (no net) -> /Bottom_Board/MOTOR_3A
- J1 pad 14: (no net) -> /Bottom_Board/T+
- J1 pad 15: (no net) -> GNDPWR
- J1 pad 2: (no net) -> GNDPWR
- J1 pad 20: (no net) -> /Bottom_Board/MOTOR_2C
- J1 pad 21: (no net) -> /Bottom_Board/MOTOR_2B
- J1 pad 22: (no net) -> /Bottom_Board/MOTOR_2A
- J1 pad 23: (no net) -> /Bottom_Board/MOTOR_1C
- J1 pad 24: (no net) -> /Bottom_Board/MOTOR_1B
- J1 pad 25: (no net) -> /Bottom_Board/MOTOR_1A
- J1 pad 4: (no net) -> /Bottom_Board/LED1+
- J1 pad 5: (no net) -> /Bottom_Board/LED1-
- J1 pad 6: (no net) -> /Bottom_Board/LED2+
- J1 pad 7: (no net) -> /Bottom_Board/LED2-
- J1 pad 8: (no net) -> /Bottom_Board/MOTOR_4C
- J1 pad 9: (no net) -> /Bottom_Board/MOTOR_4B
- P1 pad 1: Net-(P1-Pad1) -> /Upper_Board/CH7
- P1 pad 2: Net-(P1-Pad2) -> /Upper_Board/CH8
- P1 pad 3: Net-(P1-Pad3) -> /Upper_Board/CH9
- P1 pad 4: Net-(P1-Pad4) -> /Upper_Board/CH10
- P10 pad 1: (no net) -> /Bottom_Board/5V
- P10 pad 2: (no net) -> /Bottom_Board/5V
- P11 pad 1: GNDD -> /Upper_Board/U_GND
- P11 pad 2: GNDD -> /Upper_Board/D14
- P12 pad 1: /Bottom_Board/5V -> GNDPWR
- P12 pad 2: /Bottom_Board/5V -> /Bottom_Board/PWR_SW
- P13 pad 1: (no net) -> /Upper_Board/U_GND
- P13 pad 2: (no net) -> /Upper_Board/CH6
- P13 pad 3: (no net) -> /Upper_Board/CH5
- P13 pad 4: (no net) -> /Upper_Board/CH4
- P13 pad 5: (no net) -> /Upper_Board/CH3
- P13 pad 6: (no net) -> /Upper_Board/CH2
- P13 pad 7: (no net) -> /Upper_Board/CH1
- P14 pad 1: (no net) -> /Upper_Board/U_GND
- P14 pad 2: /Bottom_Board/D- -> /Upper_Board/SCL_3V3
- P14 pad 3: /Bottom_Board/D+ -> /Upper_Board/SDA_3V3
- P14 pad 4: GNDD -> /Upper_Board/3V3
- P2 pad 1: /Bottom_Board/5V -> /Upper_Board/5V
- P2 pad 2: /Bottom_Board/5V -> /Upper_Board/5V
- P2 pad 3: /Bottom_Board/5V -> /Upper_Board/5V
- P2 pad 4: /Bottom_Board/5V -> /Upper_Board/5V
- P3 pad 1: GND -> /Upper_Board/U_GND
- P3 pad 2: /5V -> /Upper_Board/D25
- P3 pad 3: /5V -> /Upper_Board/D26
- P4 pad 2: GNDD -> GNDPWR
- P6 pad 2: /Bottom_Board/3V3 -> /Upper_Board/3V3
- P7 pad 1: GNDD -> /Upper_Board/U_GND
- P7 pad 2: GNDD -> /Upper_Board/U_GND
- P7 pad 3: GNDD -> /Upper_Board/U_GND
- P7 pad 4: GNDD -> /Upper_Board/U_GND
- P8 pad 1: /Bottom_Board/5V -> /Upper_Board/5V
- P8 pad 2: /Bottom_Board/D- -> /Upper_Board/D-
- P8 pad 3: /Bottom_Board/D+ -> /Upper_Board/D+
- P8 pad 4: GNDD -> /Upper_Board/U_GND
- P9 pad 1: (no net) -> /Upper_Board/5V
- P9 pad 2: (no net) -> /Upper_Board/5V
- Q1 pad 1: /Bottom_Board/SW -> /Bottom_Board/PWR_SW
- Q1 pad 2: GNDD -> GNDPWR
- Q2 pad 2: /Bottom_Board/3V3 -> /Upper_Board/3V3
- Q3 pad 1: /Bottom_Board/3V3 -> /Upper_Board/3V3
- Q3 pad 2: /Bottom_Board/SDA_3V3 -> /Upper_Board/SDA_3V3
- Q4 pad 1: /Bottom_Board/3V3 -> /Upper_Board/3V3
- Q4 pad 2: /Bottom_Board/SCL_3V3 -> /Upper_Board/SCL_3V3
- R14 pad 1: /Bottom_Board/3V3 -> /Upper_Board/3V3
- R14 pad 2: /Bottom_Board/SDA_3V3 -> /Upper_Board/SDA_3V3
- R15 pad 1: /Bottom_Board/5V -> /Upper_Board/5V
- R16 pad 1: /Bottom_Board/3V3 -> /Upper_Board/3V3
- R16 pad 2: /Bottom_Board/SCL_3V3 -> /Upper_Board/SCL_3V3
- R17 pad 1: /Bottom_Board/5V -> /Upper_Board/5V
- R18 pad 2: GNDD -> /Upper_Board/U_GND
- R19 pad 1: GNDD -> /Upper_Board/U_GND
- R20 pad 1: /Bottom_Board/3V3 -> /Upper_Board/3V3
- R21 pad 2: /Bottom_Board/3V3 -> /Upper_Board/3V3
- R23 pad 1: /Bottom_Board/D- -> /Upper_Board/D-
- R24 pad 1: /Bottom_Board/D+ -> /Upper_Board/D+
- R3 pad 2: GNDD -> /Upper_Board/U_GND
- R6 pad 1: /Bottom_Board/V_BAT -> /Upper_Board/V_BAT+
- R6 pad 2: /Bottom_Board/ADC -> /Upper_Board/ADC
- R7 pad 1: /Bottom_Board/ADC -> /Upper_Board/ADC
- R7 pad 2: GNDD -> /Upper_Board/U_GND
- R8 pad 2: GNDD -> /Upper_Board/U_GND
- R9 pad 1: /Bottom_Board/SW -> /Bottom_Board/PWR_SW
- R9 pad 2: GNDD -> GNDPWR
- RP1 pad 5: /Bottom_Board/CH4 -> /Upper_Board/CH1
- RP1 pad 6: /Bottom_Board/CH3 -> /Upper_Board/CH2
- RP1 pad 7: /Bottom_Board/CH2 -> /Upper_Board/CH3
- RP1 pad 8: /Bottom_Board/CH1 -> /Upper_Board/CH4
- RP2 pad 1: Net-(RP2-Pad1) -> (no net)
- RP2 pad 2: Net-(RP2-Pad2) -> (no net)
- RP2 pad 5: Net-(P1-Pad2) -> /Upper_Board/CH5
- RP2 pad 6: Net-(P1-Pad1) -> /Upper_Board/CH6
- RP2 pad 7: /Bottom_Board/CH6 -> (no net)
- RP2 pad 8: /Bottom_Board/CH5 -> (no net)
- RP3 pad 5: Net-(P1-Pad6) -> /Upper_Board/CH10
- RP3 pad 6: Net-(P1-Pad5) -> /Upper_Board/CH9
- RP3 pad 7: Net-(P1-Pad4) -> /Upper_Board/CH8
- RP3 pad 8: Net-(P1-Pad3) -> /Upper_Board/CH7
- SW1 pad 1: GNDD -> /Upper_Board/U_GND
- U1 pad 1: GND -> /Upper_Board/U_GND
- U1 pad 3: /5V -> /Upper_Board/5V
- U10 pad 4: GNDD -> GNDPWR
- U11 pad 1: GNDD -> /Upper_Board/U_GND
- U11 pad 2: /Bottom_Board/3V3 -> /Upper_Board/3V3
- U11 pad 3: /Bottom_Board/5V -> /Upper_Board/5V
- U11 pad 4: /Bottom_Board/3V3 -> /Upper_Board/3V3
- U12 pad 18: (no net) -> /Upper_Board/ADC
- U12 pad 2: (no net) -> /Upper_Board/D14
- U12 pad 20: GNDD -> /Upper_Board/U_GND
- U12 pad 23: GNDD -> /Upper_Board/U_GND
- U12 pad 24: /Bottom_Board/3V3 -> /Upper_Board/3V3
- U12 pad 30: (no net) -> /Upper_Board/D26
- U12 pad 31: (no net) -> /Upper_Board/D25
- U12 pad 35: GNDD -> /Upper_Board/U_GND
- U12 pad 36: /Bottom_Board/3V3 -> /Upper_Board/3V3
- U12 pad 42: /Bottom_Board/SCL_3V3 -> /Upper_Board/SCL_3V3
- U12 pad 43: /Bottom_Board/SDA_3V3 -> /Upper_Board/SDA_3V3
- U12 pad 47: GNDD -> /Upper_Board/U_GND
- U12 pad 48: /Bottom_Board/3V3 -> /Upper_Board/3V3
- U12 pad 8: GNDD -> /Upper_Board/U_GND
- U12 pad 9: /Bottom_Board/3V3 -> /Upper_Board/3V3
- U13 pad 10: Net-(RP2-Pad1) -> Net-(RP2-Pad4)
- U13 pad 11: Net-(RP2-Pad2) -> Net-(RP2-Pad3)
- U13 pad 12: Net-(RP2-Pad3) -> (no net)
- U13 pad 13: Net-(RP2-Pad4) -> (no net)
- U13 pad 14: GNDD -> /Upper_Board/U_GND
- U13 pad 25: GNDD -> /Upper_Board/U_GND
- U13 pad 28: /Bottom_Board/5V -> /Upper_Board/5V
- U13 pad 6: Net-(RP1-Pad1) -> Net-(RP1-Pad4)
- U13 pad 7: Net-(RP1-Pad2) -> Net-(RP1-Pad3)
- U13 pad 8: Net-(RP1-Pad3) -> Net-(RP1-Pad2)
- U13 pad 9: Net-(RP1-Pad4) -> Net-(RP1-Pad1)
- U6 pad GND: GND -> /Upper_Board/U_GND
- U6 pad T_+: /T+ -> /Upper_Board/T+
- U6 pad T_-: /T- -> /Upper_Board/T-
- X1 pad 3: GNDD -> /Upper_Board/U_GND
Routing:
- net GNDPWR: track 0.00 -> 357.3 mm, vias 0 -> 14
- net /Upper_Board/5V: track 0.00 -> 227.1 mm, vias 0 -> 7
- net /Upper_Board/3V3: track 0.00 -> 205.3 mm, vias 0 -> 6
- net /Bottom_Board/V_BAT: track 0.00 -> 157.0 mm
- net /Bottom_Board/V_PWR: track 0.00 -> 98.9 mm
- net /Bottom_Board/LED2+: track 0.00 -> 87.0 mm
- net /Bottom_Board/LED2-: track 0.00 -> 82.6 mm
- net /Bottom_Board/T+: track 0.00 -> 71.7 mm
- net /Bottom_Board/LED1+: track 0.00 -> 70.1 mm
- net /Bottom_Board/MOTOR_2C: track 0.00 -> 69.7 mm
- net /Bottom_Board/LED1-: track 0.00 -> 68.4 mm
- net /Bottom_Board/CH1: track 0.00 -> 67.6 mm
- net /Bottom_Board/MOTOR_2A: track 0.00 -> 61.6 mm
- net /Bottom_Board/MOTOR_4C: track 0.00 -> 60.4 mm
- net /Upper_Board/D+: track 0.00 -> 59.2 mm
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- added copper zone on F.Cu, net /Bottom_Board/LED1+
- added copper zone on F.Cu, net /Bottom_Board/LED1-
- added copper zone on F.Cu, net /Bottom_Board/LED2+
- added copper zone on F.Cu, net /Bottom_Board/LED2-
- added copper zone on B.Cu, net /Bottom_Board/MOTOR_1A
- added copper zone on F.Cu, net /Bottom_Board/MOTOR_1A
- added copper zone on B.Cu, net /Bottom_Board/MOTOR_1B
- added copper zone on F.Cu, net /Bottom_Board/MOTOR_1B
- added copper zone on B.Cu, net /Bottom_Board/MOTOR_1C
- added copper zone on F.Cu, net /Bottom_Board/MOTOR_1C
- added copper zone on B.Cu, net /Bottom_Board/MOTOR_2A
- added copper zone on F.Cu, net /Bottom_Board/MOTOR_2A
- added copper zone on B.Cu, net /Bottom_Board/MOTOR_2B
- added copper zone on F.Cu, net /Bottom_Board/MOTOR_2B
- added copper zone on B.Cu, net /Bottom_Board/MOTOR_2C
- added copper zone on F.Cu, net /Bottom_Board/MOTOR_2C
- added copper zone on B.Cu, net /Bottom_Board/MOTOR_3A
- added copper zone on F.Cu, net /Bottom_Board/MOTOR_3A
- added copper zone on B.Cu, net /Bottom_Board/MOTOR_3B
- added copper zone on F.Cu, net /Bottom_Board/MOTOR_3B
- added copper zone on B.Cu, net /Bottom_Board/MOTOR_3C
- added copper zone on F.Cu, net /Bottom_Board/MOTOR_3C
- added copper zone on B.Cu, net /Bottom_Board/MOTOR_4A
- added copper zone on F.Cu, net /Bottom_Board/MOTOR_4A
- added copper zone on B.Cu, net /Bottom_Board/MOTOR_4B
- added copper zone on F.Cu, net /Bottom_Board/MOTOR_4B
- added copper zone on B.Cu, net /Bottom_Board/MOTOR_4C
- added copper zone on F.Cu, net /Bottom_Board/MOTOR_4C
- added copper zone on F.Cu, net /Bottom_Board/V_BAT
- added copper zone on F.Cu, net /Bottom_Board/V_PWR
- added copper zone on B.Cu, net /Upper_Board/5V
- added copper zone on F.Cu, net /Upper_Board/5V
- added copper zone on B.Cu, net /Upper_Board/U_GND
- added copper zone on F.Cu, net /Upper_Board/U_GND
- added copper zone on B.Cu, net GNDPWR
- added copper zone on F.Cu, net GNDPWR
- added copper zone on F.Cu, net Net-(D3-Pad2)
- added copper zone on F.Cu, net Net-(D4-Pad2)
Other:
- board size 99 x 70 mm -> 190 x 72 mm
- net class Default: clearance 0.2 -> 0.12; trace_width 2 -> 0.5
- rule trace_clearance: 0.2 -> 0.12
- board text added: "10"
- board text added: "3V3"
- board text added: "5V"
- board text added: "7"
- board text added: "8"
- board text added: "9"
- board text added: "AUX I2C"
- board text added: "BAT+"
- board text added: "BOOT 0"
- board text added: "CH"
- board text added: "Connection"
- board text added: "DFU"
- board text added: "Ethernet"
- board text added: "Extra PWM"
- board text added: "GND"
- board text added: "GND 6 5 4 3 2 1"
- board text added: "GND D+ D- 5V"
- board text added: "GND RX1 TX1"
- board text added: "GND T- T+"
- board text added: "LED DRIVER 1"
- board text added: "LED DRIVER 2"
- board text added: "MCU State"
- board text added: "PWM"
- board text added: "PWR SW"
- board text added: "SCL"
- board text added: "SDA"
- board text added: "V+"
- board text added: "V-"
