File: Main_Board/Main_Board.kicad_pcb (KiCad board)
At the start: 2 copper layers, 190 x 72 mm, 95 parts, among them J1 DB25, P1 CONN_01X04, P10 CONN_01X02, P11 CONN_01X03, P12 CONN_01X03, P13 CONN_01X07, P14 CONN_01X04, P15 CONN_01X07, P16 CONN_01X03, P17 CONN_01X03, P2 CONN_01X04, P3 CONN_01X03, P4 CONN_01X02, P6 BOOT, P7 CONN_01X04, P8 CONN_01X04, P9 CONN_01X02, Q1 DMN65D8L, Q2 BSS84, Q3 BSS138, Q4 BSS138, SW1 RESET, U1 TLV1117LV33, U10 DSN-MINI-360, U11 TLV1117LV33, U12 STM32F103CBT6, U13 pca9685, U14 MPU9250, U2 DYS_mini_ESC, U3 DYS_mini_ESC, U4 DYS_mini_ESC, U5 DYS_mini_ESC, U6 TENDA_P200, U7 AL8805W5, U8 AL8805W5, U9 SI4425DDY, X1 8MHz

Commit message: Schematic arrangement
Other:
- net class Default: trace_width 0.5 -> 0.25
Changed lines of the file:
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@@
     (links 287)
     (no_connects 0)
-    (area 159.924999 67.924999 240.075001 132.075001)
+    (area 49.924999 63.924999 240.075001 136.075001)
     (thickness 1.6)
     (drawings 63)
@@
   )
   (setup
-    (last_trace_width 0.5)
+    (last_trace_width 0.25)
     (trace_clearance 0.12)
     (zone_clearance 0.508)
@@
     (visible_elements 7FFFEF7F)
     (pcbplotparams
-      (layerselection 0x00030_80000001)
+      (layerselection 0x010f0_80000001)
       (usegerberextensions false)
       (excludeedgelayer true)
@@
       (outputformat 1)
       (mirror false)
-      (drillshape 1)
+      (drillshape 0)
       (scaleselection 1)
-      (outputdirectory ""))
+      (outputdirectory C:/Users/YJ/Desktop/Main_Baord/))
   )
   (net 0 "")
@@
   (net_class Default "This is the default net class."
     (clearance 0.12)
-    (trace_width 0.5)
+    (trace_width 0.25)
     (via_dia 0.6)
     (via_drill 0.4)
@@
   (segment (start 168.75 93.25) (end 164.89902 93.25) (width 0.3) (layer F.Cu) (net 2))
   (segment (start 183.36 96.58) (end 181.94 98) (width 0.3) (layer F.Cu) (net 3))
-  (segment (start 181.94 98) (end 171.45 98) (width 0.3) (layer F.Cu) (net 3))
-  (segment (start 171.45 98) (end 170.95 97.5) (width 0.3) (layer F.Cu) (net 3))
   (segment (start 170.95 97.5) (end 170.25 97.5) (width 0.3) (layer F.Cu) (net 3))
+  (segment (start 171.45 98) (end 170.95 97.5) (width 0.3) (layer F.Cu) (net 3))
+  (segment (start 181.94 98) (end 171.45 98) (width 0.3) (layer F.Cu) (net 3))
   (segment (start 174.33 96.58) (end 171 93.25) (width 0.3) (layer F.Cu) (net 4))
   (segment (start 171 93.25) (end 170.25 93.25) (width 0.3) (layer F.Cu) (net 4))
@@
   (segment (start 213.671024 88.499004) (end 215.650996 88.499004) (width 0.25) (layer F.Cu) (net 61))
   (segment (start 215.650996 88.499004) (end 217.4 86.75) (width 0.25) (layer F.Cu) (net 61))
+  (segment (start 194.026108 94.07943) (end 194.026108 87.47543) (width 1) (layer F.Cu) (net 62))
   (segment (start 163.5 91.25) (end 162.80098 91.94902) (width 0.5) (layer F.Cu) (net 62))
   (segment (start 162.80098 91.94902) (end 162.80098 93.25) (width 0.5) (layer F.Cu) (net 62))
@@
   (segment (start 194.026108 87.47543) (end 194.838908 87.47543) (width 0.5) (layer F.Cu) (net 62))
   (segment (start 185.9 96.58) (end 185.9 99.12) (width 1) (layer F.Cu) (net 62))
-  (segment (start 194.026108 94.07943) (end 194.026108 87.47543) (width 1) (layer F.Cu) (net 62))
   (segment (start 194.026108 97.12743) (end 194.026108 94.07943) (width 1) (layer F.Cu) (net 62))
   (segment (start 189.75 75.75) (end 189.075 76.425) (width 0.3) (layer F.Cu) (net 63))
@@
   (segment (start 228.583334 70.305248) (end 227.811554 70.305248) (width 0.3) (layer F.Cu) (net 64))
   (segment (start 227.811554 70.305248) (end 227.061554 71.055248) (width 0.3) (layer F.Cu) (net 64))
+  (segment (start 233.15 78.15) (end 233.15 77.35) (width 0.25) (layer F.Cu) (net 65))
+  (segment (start 233.15 77.35) (end 233.5 77) (width 0.25) (layer F.Cu) (net 65))
+  (segment (start 180.82 99.12) (end 178.88 99.12) (width 0.5) (layer F.Cu) (net 65))
   (via (at 230.25 80.25) (size 0.6) (drill 0.4) (layers F.Cu B.Cu) (net 65))
   (segment (start 229.1 80.015) (end 230.015 80.015) (width 0.2) (layer F.Cu) (net 65))
@@
   (segment (start 224.965 79.215) (end 224.75 79) (width 0.2) (layer F.Cu) (net 65))
   (via (at 224.75 79) (size 0.6) (drill 0.4) (layers F.Cu B.Cu) (net 65))
-  (segment (start 180.82 99.12) (end 178.88 99.12) (width 0.5) (layer F.Cu) (net 65))
   (segment (start 182.15 84.225) (end 181.275 84.225) (width 0.5) (layer F.Cu) (net 65))
   (segment (start 181.275 84.225) (end 180.75 84.75) (width 0.5) (layer F.Cu) (net 65))
@@
   (segment (start 189.225 77.725) (end 190 78.5) (width 0.5) (layer F.Cu) (net 65))
   (via (at 190 78.5) (size 0.6) (drill 0.4) (layers F.Cu B.Cu) (net 65))
-  (segment (start 233.15 78.15) (end 233.15 77.35) (width 0.25) (layer F.Cu) (net 65))
-  (segment (start 233.15 77.35) (end 233.5 77) (width 0.25) (layer F.Cu) (net 65))
   (via (at 233.5 77) (size 0.6) (drill 0.4) (layers F.Cu B.Cu) (net 65))
   (segment (start 232.75 82.5) (end 232.75 83.25) (width 0.25) (layer B.Cu) (net 65))
