File: Main_Board/Main_Board.sch (KiCad schematic (older format))
At the start: 20 parts, among them P1 CONN_02X04, P2 CONN_02X04, P3 CONN_01X03, P5 CONN_02X12, U1 TLV1117LV33, U2 DYS_mini_ESC, U3 DYS_mini_ESC, U4 DYS_mini_ESC, U5 DYS_mini_ESC, U6 TENDA_P200

Commit message: Main Board update
Parts:
- P5: footprint (none) -> KiCad_Footprint:Socket_Strip_Angled_2x12
Changed lines of the file:
@@
 LIBS:valves
 LIBS:custom_lib
+LIBS:Main_Board-cache
 EELAYER 25 0
 EELAYER END
@@
 F 0 "P5" H 3875 3325 50  0000 C CNN
 F 1 "CONN_02X12" V 3875 2775 50  0000 C CNN
-F 2 "" H 3875 1575 50  0000 C CNN
+F 2 "KiCad_Footprint:Socket_Strip_Angled_2x12" H 3875 1575 50  0001 C CNN
 F 3 "" H 3875 1575 50  0000 C CNN
 	1    3875 2775

Commit message: Main Board : Add Braket Hole
Parts:
- P1, P2: value CONN_02X04 -> CONN_01X08; footprint Socket_Strips:Socket_Strip_Straight_2x04 -> Socket_Strips:Socket_Strip_Straight_1x08; symbol CONN_02X04 -> CONN_01X08
Other:
- moved on the sheet: P3
Changed lines of the file:
@@
 3V3
 $Comp
-L CONN_02X04 P1
+L CONN_01X08 P1
 U 1 1 5828C2FF
-P 3800 4775
-F 0 "P1" H 3800 5025 50  0000 C CNN
-F 1 "CONN_02X04" H 3800 4525 50  0000 C CNN
-F 2 "Socket_Strips:Socket_Strip_Straight_2x04" H 3800 3575 50  0001 C CNN
-F 3 "" H 3800 3575 50  0000 C CNN
-	1    3800 4775
+P 2175 4850
+F 0 "P1" H 2175 5100 50  0000 C CNN
+F 1 "CONN_01X08" V 2300 4825 50  0000 C CNN
+F 2 "Socket_Strips:Socket_Strip_Straight_1x08" H 2175 3650 50  0001 C CNN
+F 3 "" H 2175 3650 50  0000 C CNN
+	1    2175 4850
 	1    0    0    -1
 $EndComp
@@
 L GND #PWR08
 U 1 1 5828C6C6
-P 4325 4625
-F 0 "#PWR08" H 4325 4375 50  0001 C CNN
-F 1 "GND" H 4325 4475 50  0000 C CNN
-F 2 "" H 4325 4625 50  0000 C CNN
-F 3 "" H 4325 4625 50  0000 C CNN
-	1    4325 4625
-	0    -1   -1   0
-$EndComp
-Text Label 3225 4625 0    60   Italic 0
+P 1700 5200
+F 0 "#PWR08" H 1700 4950 50  0001 C CNN
+F 1 "GND" H 1700 5050 50  0000 C CNN
+F 2 "" H 1700 5200 50  0000 C CNN
+F 3 "" H 1700 5200 50  0000 C CNN
+	1    1700 5200
+	0    1    1    0
+$EndComp
+Text Label 1650 4500 0    60   Italic 0
 V_BAT
-Text Label 3225 4725 0    60   ~ 0
+Text Label 1650 4600 0    60   ~ 0
 CH1
-Text Label 4150 4725 0    60   ~ 0
+Text Label 1875 5100 2    60   ~ 0
 CH2
-Text Label 3225 4825 0    60   ~ 0
+Text Label 1650 4700 0    60   ~ 0
 CH3
-Text Label 4150 4825 0    60   ~ 0
+Text Label 1875 5000 2    60   ~ 0
 CH4
-Text Label 3225 4925 0    60   ~ 0
+Text Label 1650 4800 0    60   ~ 0
 CH5
-Text Label 4150 4925 0    60   ~ 0
+Text Label 1875 4900 2    60   ~ 0
 CH6
-Text Notes 3325 4400 0    60   Italic 0
+Text Notes 1575 4325 0    60   Italic 0
 CH1 : ESC 1\nCH2 : ESC 2\nCH3 : ESC 3\nCH4 : ESC 4\nCH5 : LED DRIVER 1\nCH6 : LED DRIVER 2
 $Comp
 L CONN_01X03 P3
 U 1 1 5828FD4F
-P 4100 6475
-F 0 "P3" H 4100 6675 50  0000 C CNN
-F 1 "CONN_01X03" V 4200 6475 50  0000 C CNN
-F 2 "Socket_Strips:Socket_Strip_Straight_1x03" H 4100 6475 50  0001 C CNN
-F 3 "" H 4100 6475 50  0000 C CNN
-	1    4100 6475
-	1    0    0    -1
-$EndComp
-Text Label 3400 6475 0    60   ~ 0
+P 3400 5825
+F 0 "P3" H 3400 6025 50  0000 C CNN
+F 1 "CONN_01X03" V 3500 5825 50  0000 C CNN
+F 2 "Socket_Strips:Socket_Strip_Straight_1x03" H 3400 5825 50  0001 C CNN
+F 3 "" H 3400 5825 50  0000 C CNN
+	1    3400 5825
+	1    0    0    -1
+$EndComp
+Text Label 2700 5825 0    60   ~ 0
 5V
-Text Label 3400 6575 0    60   ~ 0
+Text Label 2700 5925 0    60   ~ 0
 5V
 $Comp
 L GND #PWR09
 U 1 1 582905C9
-P 3700 6375
-F 0 "#PWR09" H 3700 6125 50  0001 C CNN
-F 1 "GND" H 3700 6225 50  0000 C CNN
-F 2 "" H 3700 6375 50  0000 C CNN
-F 3 "" H 3700 6375 50  0000 C CNN
-	1    3700 6375
+P 3000 5725
+F 0 "#PWR09" H 3000 5475 50  0001 C CNN
+F 1 "GND" H 3000 5575 50  0000 C CNN
+F 2 "" H 3000 5725 50  0000 C CNN
+F 3 "" H 3000 5725 50  0000 C CNN
+	1    3000 5725
 	0    1    1    0
 $EndComp
-Text Notes 3350 6150 0    60   Italic 0
+Text Notes 2650 6200 0    60   Italic 0
 Raspberry Pi Power
 Text Label 2700 925  0    60   ~ 0
@@
 $EndComp
 $Comp
-L CONN_02X04 P2
+L CONN_01X08 P2
 U 1 1 58293B03
-P 3800 5500
-F 0 "P2" H 3800 5750 50  0000 C CNN
-F 1 "CONN_02X04" H 3800 5250 50  0000 C CNN
-F 2 "Socket_Strips:Socket_Strip_Straight_2x04" H 3800 4300 50  0001 C CNN
-F 3 "" H 3800 4300 50  0000 C CNN
-	1    3800 5500
-	1    0    0    -1
-$EndComp
-Text Label 4175 5350 0    60   ~ 0
+P 3400 4900
+F 0 "P2" H 3400 5150 50  0000 C CNN
+F 1 "CONN_01X08" V 3525 4875 50  0000 C CNN
+F 2 "Socket_Strips:Socket_Strip_Straight_1x08" H 3400 3700 50  0001 C CNN
+F 3 "" H 3400 3700 50  0000 C CNN
+	1    3400 4900
+	1    0    0    -1
+$EndComp
+Text Label 3075 4950 2    60   ~ 0
 SCL
-Text Label 4175 5450 0    60   ~ 0
+Text Label 3075 5050 2    60   ~ 0
 SDA
-Text Label 4125 5550 0    60   ~ 0
+Text Label 3125 5150 2    60   ~ 0
 ADC1
 $Comp
 L GND #PWR010
 U 1 1 582941F8
-P 4225 5650
-F 0 "#PWR010" H 4225 5400 50  0001 C CNN
-F 1 "GND" H 4225 5500 50  0000 C CNN
-F 2 "" H 4225 5650 50  0000 C CNN
-F 3 "" H 4225 5650 50  0000 C CNN
-	1    4225 5650
-	0    -1   -1   0
-$EndComp
-NoConn ~ 3550 5450
-NoConn ~ 3550 5550
-NoConn ~ 3550 5650
-Text Label 3150 5350 0    60   ~ 0
+P 3025 5250
+F 0 "#PWR010" H 3025 5000 50  0001 C CNN
+F 1 "GND" H 3025 5100 50  0000 C CNN
+F 2 "" H 3025 5250 50  0000 C CNN
+F 3 "" H 3025 5250 50  0000 C CNN
+	1    3025 5250
+	0    1    -1   0
+$EndComp
+NoConn ~ 3200 4650
+NoConn ~ 3200 4750
+NoConn ~ 3200 4850
+Text Label 2800 4550 0    60   ~ 0
 PWR_SW
 Wire Wire Line
@@
 	4575 1425 4575 1350
 Wire Wire Line
-	3550 4625 3225 4625
-Wire Wire Line
-	4050 4625 4325 4625
-Wire Wire Line
-	3550 4725 3225 4725
-Wire Wire Line
-	4050 4725 4325 4725
-Wire Wire Line
-	3550 4825 3225 4825
-Wire Wire Line
-	3550 4925 3225 4925
-Wire Wire Line
-	4050 4825 4325 4825
-Wire Wire Line
-	4050 4925 4325 4925
-Wire Wire Line
-	3900 6475 3400 6475
-Wire Wire Line
-	3900 6575 3400 6575
-Wire Wire Line
-	3700 6375 3900 6375
-Wire Wire Line
-	4050 5350 4325 5350
-Wire Wire Line
-	4050 5450 4325 5450
-Wire Wire Line
-	4050 5550 4325 5550
-Wire Wire Line
-	4050 5650 4225 5650
-Wire Wire Line
-	3150 5350 3550 5350
+	1975 4500 1650 4500
+Wire Wire Line
+	1975 5200 1700 5200
+Wire Wire Line
+	1975 4600 1650 4600
+Wire Wire Line
+	1975 5100 1700 5100
+Wire Wire Line
+	1975 4700 1650 4700
+Wire Wire Line
+	1975 4800 1650 4800
+Wire Wire Line
+	1975 5000 1700 5000
+Wire Wire Line
+	1975 4900 1700 4900
+Wire Wire Line
+	3200 5825 2700 5825
+Wire Wire Line
+	3200 5925 2700 5925
+Wire Wire Line
+	3000 5725 3200 5725
+Wire Wire Line
+	3200 4950 2925 4950
+Wire Wire Line
+	3200 5050 2925 5050
+Wire Wire Line
+	3200 5150 2925 5150
+Wire Wire Line
+	3200 5250 3025 5250
+Wire Wire Line
+	2800 4550 3200 4550
 Wire Wire Line
 	3625 2225 3075 2225

Commit message: Main Board incomplete routing
Connections:
- net labels added: 3V3_Front, ADC, BOOT, SW
- net labels removed: ADC1, PWR_SW
- wire segments 85 -> 88
- no-connect marks 5 -> 2
Other:
- note added: "Left Braket"
- note added: "Righit Braket"
- moved on the sheet: P1, P2, P3

Commit message: Main Board : Separate PCB into two part
Parts:
- removed C3, C4, C5, C6: CP1, Capacitors_SMD:c_elec_6.3x4.5, symbol CP1
- removed P1, P2: CONN_01X08, Socket_Strips:Socket_Strip_Straight_1x08, symbol CONN_01X08
- removed P5: CONN_02X12, KiCad_Footprint:Socket_Strip_Angled_2x12, symbol CONN_02X12
- removed U2, U3, U4, U5: DYS_mini_ESC, KiCad_Footprint:DYS_Mini_ESC, symbol DYS_mini_ESC
- added J1: DB25, Connect:DB25FC, symbol DB25
Connections:
- net labels removed: 3V3_Front, ADC, BOOT, CH1, CH2, CH3, CH4, CH5, CH6, MOTOR_1A, MOTOR_1B, MOTOR_1C, MOTOR_2A, MOTOR_2B, MOTOR_2C, MOTOR_3A, MOTOR_3B, MOTOR_3C, MOTOR_4A, MOTOR_4B, MOTOR_4C, SCL, SDA, SW, V_BAT
- wire segments 88 -> 23
Other:
- note removed: "CH1 : ESC 1\nCH2 : ESC 2\nCH3 : ESC 3\nCH4 : ESC 4\nCH5 : LED DRIVER 1\nCH6 : LED DRIVER 2"
- note removed: "Left Braket"
- note removed: "Righit Braket"

Commit message: shit
Changed lines of the file:
@@
 NoConn ~ 8200 4900
 $Comp
-L GND #PWR01
+L GND #PWR4
 U 1 1 58286916
 P 6275 4400
-F 0 "#PWR01" H 6275 4150 50  0001 C CNN
+F 0 "#PWR4" H 6275 4150 50  0001 C CNN
 F 1 "GND" H 6275 4250 50  0000 C CNN
 F 2 "" H 6275 4400 50  0000 C CNN
@@
 $EndComp
 $Comp
-L GND #PWR02
+L GND #PWR3
 U 1 1 5828754C
 P 5325 4800
-F 0 "#PWR02" H 5325 4550 50  0001 C CNN
+F 0 "#PWR3" H 5325 4550 50  0001 C CNN
 F 1 "GND" H 5325 4650 50  0000 C CNN
 F 2 "" H 5325 4800 50  0000 C CNN
@@
 $EndComp
 $Comp
-L GND #PWR03
+L GND #PWR1
 U 1 1 58289EFC
 P 3775 1475
-F 0 "#PWR03" H 3775 1225 50  0001 C CNN
+F 0 "#PWR1" H 3775 1225 50  0001 C CNN
 F 1 "GND" H 3775 1325 50  0000 C CNN
 F 2 "" H 3775 1475 50  0000 C CNN
@@
 5V
 $Comp
-L GND #PWR04
+L GND #PWR2
 U 1 1 582905C9
 P 3800 6900
-F 0 "#PWR04" H 3800 6650 50  0001 C CNN
+F 0 "#PWR2" H 3800 6650 50  0001 C CNN
 F 1 "GND" H 3800 6750 50  0000 C CNN
 F 2 "" H 3800 6900 50  0000 C CNN
@@
 $EndComp
 $Sheet
-S 9500 1100 1275 2325
+S 7425 750  1275 2325
 U 582D6DEA
 F0 "Bottom_Board" 60
 F1 "Bottom_Board.sch" 60
-F2 "L_GND" I L 9500 1925 60
+F2 "L_GND" I L 7425 1575 60
 $EndSheet
 $EndSCHEMATC

Commit message: Final Routing
Parts:
- removed C1: C, Capacitors_SMD:C_0805, symbol C
- removed C2: C, Capacitors_SMD:C_0603, symbol C
- removed D1, D2: LED, LEDs:LED_0805, symbol LED
- removed J1: DB25, Connect:DB25FC, symbol DB25
- removed P3: CONN_01X03, Socket_Strips:Socket_Strip_Straight_1x03, symbol CONN_01X03
- removed R1, R2: 330, Capacitors_SMD:C_0603, symbol R
- removed U1: TLV1117LV33, TO_SOT_Packages_SMD:SOT-223, symbol TLV1117LV33
- removed U6: TENDA_P200, KiCad_Footprint:Tenda_p200, symbol TENDA_P200
Connections:
- net labels removed: 3V3, 5V, GND, T+, T-
- wire segments 23 -> 0
- no-connect marks 2 -> 0
Other:
- note removed: "Raspberry Pi Power"
Changed lines of the file:
@@
 $Descr A4 11693 8268
 encoding utf-8
-Sheet 1 2
+Sheet 1 3
 Title ""
 Date ""
@@
 Comment4 ""
 $EndDescr
-$Comp
-L TENDA_P200 U6
-U 1 1 582866B6
-P 7350 5050
-F 0 "U6" H 7750 4900 60  0000 C CNN
-F 1 "TENDA_P200" H 6950 6100 60  0000 C CNN
-F 2 "KiCad_Footprint:Tenda_p200" H 7350 4800 60  0001 C CNB
-F 3 "" H 7350 5050 60  0000 C CNN
-	1    7350 5050
-	1    0    0    -1
-$EndComp
-NoConn ~ 8200 4900
-$Comp
-L GND #PWR4
-U 1 1 58286916
-P 6275 4400
-F 0 "#PWR4" H 6275 4150 50  0001 C CNN
-F 1 "GND" H 6275 4250 50  0000 C CNN
-F 2 "" H 6275 4400 50  0000 C CNN
-F 3 "" H 6275 4400 50  0000 C CNN
-	1    6275 4400
-	0    1    1    0
-$EndComp
-Text Label 5850 4200 0    60   ~ 0
-3V3
-Text Label 8575 4200 0    60   ~ 0
-T+
-NoConn ~ 6350 4600
-$Comp
-L LED D1
-U 1 1 5828739F
-P 5600 4800
-F 0 "D1" H 5600 4900 50  0000 C CNN
-F 1 "LED" H 5600 4700 50  0000 C CNN
-F 2 "LEDs:LED_0805" H 5625 5000 50  0001 C CNN
-F 3 "" H 5600 4800 50  0000 C CNN
-	1    5600 4800
-	1    0    0    -1
-$EndComp
-$Comp
-L R R1
-U 1 1 58287494
-P 6050 4800
-F 0 "R1" V 6130 4800 50  0000 C CNN
-F 1 "330" V 6050 4800 50  0000 C CNN
-F 2 "Capacitors_SMD:C_0603" V 5980 4800 50  0001 C CNN
-F 3 "" H 6050 4800 50  0000 C CNN
-	1    6050 4800
-	0    1    1    0
-$EndComp
-$Comp
-L GND #PWR3
-U 1 1 5828754C
-P 5325 4800
-F 0 "#PWR3" H 5325 4550 50  0001 C CNN
-F 1 "GND" H 5325 4650 50  0000 C CNN
-F 2 "" H 5325 4800 50  0000 C CNN
-F 3 "" H 5325 4800 50  0000 C CNN
-	1    5325 4800
-	0    1    1    0
-$EndComp
-$Comp
-L LED D2
-U 1 1 582875B3
-P 5600 5000
-F 0 "D2" H 5600 5100 50  0000 C CNN
-F 1 "LED" H 5725 5075 50  0000 C CNN
-F 2 "LEDs:LED_0805" H 5500 5225 50  0001 C CNN
-F 3 "" H 5600 5000 50  0000 C CNN
-	1    5600 5000
-	-1   0    0    1
-$EndComp
-$Comp
-L R R2
-U 1 1 582877C3
-P 6050 5000
-F 0 "R2" V 6130 5000 50  0000 C CNN
-F 1 "330" V 6050 5000 50  0000 C CNN
-F 2 "Capacitors_SMD:C_0603" V 5980 5000 50  0001 C CNN
-F 3 "" H 6050 5000 50  0000 C CNN
-	1    6050 5000
-	0    1    1    0
-$EndComp
-Text Label 5050 5000 0    60   ~ 0
-3V3
-$Comp
-L TLV1117LV33 U1
-U 1 1 58289A85
-P 3775 975
-F 0 "U1" H 3475 1225 50  0000 C CNN
-F 1 "TLV1117LV33" H 3775 1175 50  0000 C CNN
-F 2 "TO_SOT_Packages_SMD:SOT-223" H 3775 1075 50  0001 C CIN
-F 3 "" H 3775 975 50  0000 C CNN
-	1    3775 975
-	1    0    0    -1
-$EndComp
-$Comp
-L C C1
-U 1 1 58289D95
-P 3175 1200
-F 0 "C1" H 3200 1300 50  0000 L CNN
-F 1 "C" H 3200 1100 50  0000 L CNN
-F 2 "Capacitors_SMD:C_0805" H 3213 1050 50  0001 C CNN
-F 3 "" H 3175 1200 50  0000 C CNN
-	1    3175 1200
-	1    0    0    -1
-$EndComp
-$Comp
-L GND #PWR1
-U 1 1 58289EFC
-P 3775 1475
-F 0 "#PWR1" H 3775 1225 50  0001 C CNN
-F 1 "GND" H 3775 1325 50  0000 C CNN
-F 2 "" H 3775 1475 50  0000 C CNN
-F 3 "" H 3775 1475 50  0000 C CNN
-	1    3775 1475
-	1    0    0    -1
-$EndComp
-$Comp
-L C C2
-U 1 1 5828A25A
-P 4575 1200
-F 0 "C2" H 4600 1300 50  0000 L CNN
-F 1 "C" H 4600 1100 50  0000 L CNN
-F 2 "Capacitors_SMD:C_0603" H 4613 1050 50  0001 C CNN
-F 3 "" H 4575 1200 50  0000 C CNN
-	1    4575 1200
-	1    0    0    -1
-$EndComp
-Text Label 4900 925  0    60   ~ 0
-3V3
-$Comp
-L CONN_01X03 P3
-U 1 1 5828FD4F
-P 4200 7000
-F 0 "P3" H 4200 7200 50  0000 C CNN
-F 1 "CONN_01X03" V 4300 7000 50  0000 C CNN
-F 2 "Socket_Strips:Socket_Strip_Straight_1x03" H 4200 7000 50  0001 C CNN
-F 3 "" H 4200 7000 50  0000 C CNN
-	1    4200 7000
-	1    0    0    -1
-$EndComp
-Text Label 3500 7000 0    60   ~ 0
-5V
-Text Label 3500 7100 0    60   ~ 0
-5V
-$Comp
-L GND #PWR2
-U 1 1 582905C9
-P 3800 6900
-F 0 "#PWR2" H 3800 6650 50  0001 C CNN
-F 1 "GND" H 3800 6750 50  0000 C CNN
-F 2 "" H 3800 6900 50  0000 C CNN
-F 3 "" H 3800 6900 50  0000 C CNN
-	1    3800 6900
-	0    1    1    0
-$EndComp
-Text Notes 3450 7375 0    60   Italic 0
-Raspberry Pi Power
-Text Label 2700 925  0    60   ~ 0
-5V
-Text Label 8575 4400 0    60   ~ 0
-T-
-Wire Wire Line
-	6350 4400 6275 4400
-Wire Wire Line
-	6350 4200 5850 4200
-Wire Wire Line
-	8200 4200 8675 4200
-Wire Wire Line
-	8200 4400 8675 4400
-Wire Wire Line
-	6200 4800 6350 4800
-Wire Wire Line
-	5900 4800 5800 4800
-Wire Wire Line
-	5400 4800 5325 4800
-Wire Wire Line
-	6200 5000 6350 5000
-Wire Wire Line
-	5800 5000 5900 5000
-Wire Wire Line
-	5400 5000 5050 5000
-Wire Wire Line
-	3175 925  3175 1050
-Connection ~ 3175 925
-Wire Wire Line
-	3775 1275 3775 1475
-Wire Wire Line
-	3175 1350 3175 1425
-Wire Wire Line
-	3175 1425 4575 1425
-Connection ~ 3775 1425
-Wire Wire Line
-	4225 925  5050 925
-Wire Wire Line
-	4225 1075 4450 1075
-Wire Wire Line
-	4450 1075 4450 925
-Connection ~ 4450 925
-Wire Wire Line
-	4575 925  4575 1050
-Connection ~ 4575 925
-Wire Wire Line
-	4575 1425 4575 1350
-Wire Wire Line
-	4000 7000 3500 7000
-Wire Wire Line
-	4000 7100 3500 7100
-Wire Wire Line
-	3800 6900 4000 6900
-Wire Wire Line
-	3325 925  2700 925
-$Comp
-L DB25 J1
-U 1 1 582D52F2
-P 2525 3725
-F 0 "J1" H 2575 5075 50  0000 C CNN
-F 1 "DB25" H 2475 2375 50  0000 C CNN
-F 2 "Connect:DB25FC" H 2525 3725 50  0001 C CNN
-F 3 "" H 2525 3725 50  0000 C CNN
-	1    2525 3725
-	1    0    0    -1
-$EndComp
 $Sheet
 S 7425 750  1275 2325
@@
 F2 "L_GND" I L 7425 1575 60
 $EndSheet
+$Sheet
+S 5725 1925 1175 1300
+U 58347913
+F0 "Upper_Board" 60
+F1 "Upper_Board.sch" 60
+$EndSheet
 $EndSCHEMATC

Commit message: Schematic arrangement
Changed lines of the file:
@@
 $EndDescr
 $Sheet
-S 7425 750  1275 2325
+S 2200 900  1200 1300
 U 582D6DEA
 F0 "Bottom_Board" 60
 F1 "Bottom_Board.sch" 60
-F2 "L_GND" I L 7425 1575 60
 $EndSheet
 $Sheet
-S 5725 1925 1175 1300
+S 875  900  1175 1300
 U 58347913
 F0 "Upper_Board" 60
